File: PCB/dotflipper.brd (EAGLE design)
At the start: 224.8 x 107.6 mm, 391 parts, among them IC10 UDN2982, IC12 PCA9685, IC13 UDN2982, IC15 PCA9685, IC16 UDN2982, IC18 PCA9685, IC22 UDN2982, IC24 PCA9685, IC4 UDN2982, IC6 PCA9685, IC7 UDN2982, IC9 PCA9685, J3 2X6 FEMALE, Q1 BSS138, Q2 BSS138, X1 2534-, X2 2516-, X3 2516-, X4 MSTBA2, X5 MSTBA2

Commit message: Minor cleanup of schematic. Made PDFs for those without Eagle.
Parts:
- J3: value 2X6 FEMALE -> SHA BADGE
- WEMOS1: value (none) -> Wemos D1 mini
Changed lines of the file:
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@@
 <layer number="37" name="tTest" color="7" fill="1" visible="no" active="yes"/>
 <layer number="38" name="bTest" color="7" fill="1" visible="no" active="yes"/>
-<layer number="39" name="tKeepout" color="4" fill="11" visible="yes" active="yes"/>
-<layer number="40" name="bKeepout" color="1" fill="11" visible="yes" active="yes"/>
-<layer number="41" name="tRestrict" color="4" fill="10" visible="yes" active="yes"/>
-<layer number="42" name="bRestrict" color="1" fill="10" visible="yes" active="yes"/>
-<layer number="43" name="vRestrict" color="2" fill="10" visible="yes" active="yes"/>
+<layer number="39" name="tKeepout" color="4" fill="11" visible="no" active="yes"/>
+<layer number="40" name="bKeepout" color="1" fill="11" visible="no" active="yes"/>
+<layer number="41" name="tRestrict" color="4" fill="10" visible="no" active="yes"/>
+<layer number="42" name="bRestrict" color="1" fill="10" visible="no" active="yes"/>
+<layer number="43" name="vRestrict" color="2" fill="10" visible="no" active="yes"/>
 <layer number="44" name="Drills" color="7" fill="1" visible="no" active="yes"/>
 <layer number="45" name="Holes" color="7" fill="1" visible="yes" active="yes"/>
@@
 <attribute name="VALUE" x="4.318" y="59.69" size="0.6096" layer="27" font="vector" ratio="20" rot="R270"/>
 </element>
-<element name="WEMOS1" library="esp8266modules" package="WEMOS-D1-MINI" value="" x="131.191" y="20.066" smashed="yes"/>
+<element name="WEMOS1" library="esp8266modules" package="WEMOS-D1-MINI" value="Wemos D1 mini" x="131.191" y="20.066" smashed="yes"/>
 <element name="Q1" library="SparkFun-DiscreteSemi" library_urn="urn:adsk.eagle:library:514" package="SOT23-3" package3d_urn="urn:adsk.eagle:package:38446/1" value="BSS138" x="109.22" y="37.973" smashed="yes">
 <attribute name="PROD_ID" value="TRANS-00830" x="109.22" y="37.973" size="1.778" layer="27" display="off"/>
@@
 <element name="R18" library="rcl" package="R0603" value="10k" x="103.505" y="34.544" smashed="yes" rot="R180"/>
 <element name="R19" library="rcl" package="R0603" value="10k" x="103.505" y="41.783" smashed="yes"/>
-<element name="J3" library="SparkFun-Connectors" library_urn="urn:adsk.eagle:library:513" package="2X6" package3d_urn="urn:adsk.eagle:package:38277/1" value="2X6 FEMALE" x="100.33" y="13.335" smashed="yes">
+<element name="J3" library="SparkFun-Connectors" library_urn="urn:adsk.eagle:library:513" package="2X6" package3d_urn="urn:adsk.eagle:package:38277/1" value="SHA BADGE" x="100.33" y="13.335" smashed="yes">
 <attribute name="PROD_ID" value="CONN-12423" x="100.33" y="13.335" size="1.778" layer="27" display="off"/>
 </element>
