File: PCB/dotflipper.sch (EAGLE design)
At the start: 391 parts, among them IC10 UDN2982, IC12 PCA9685, IC13 UDN2982, IC15 PCA9685, IC16 UDN2982, IC18 PCA9685, IC22 UDN2982, IC24 PCA9685, IC4 UDN2982, IC6 PCA9685, IC7 UDN2982, IC9 PCA9685, J3 2X6 FEMALE, Q1 BSS138, Q2 BSS138, X1 2534-, X2 2516-, X3 2516-, X4 MSTBA2, X5 MSTBA2

Commit message: Minor cleanup of schematic. Made PDFs for those without Eagle.
Parts:
- J3: value 2X6 FEMALE -> SHA BADGE
- WEMOS1: value (none) -> Wemos D1 mini
Other:
- note added: "Schematic for Flip Dot controller github.com/sebastius/dotflipper CC-BY-SA 4.0"
- moved on the sheet: ARDUINO_NANO, C1, C10, C11, C12, C13, C14, C15, C16, C2, C3, C4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
